File: NES3.kicad_pcb (KiCad board)
At the start: 2 copper layers, 101.5 x 50.8 mm, 23 parts, among them SW1 SW_DPDT_x2, U2 27C256 - PLCC32, U3 74HC74, U4 74HC32, U5 27C256 - PLCC32, U7 HY6264ALJ

Commit message: Add files via upload
Parts:
- U2: value 27C256 - PLCC32 -> 27C256 - PLCC32 - PPU
- U5: value 27C256 - PLCC32 -> 27C256 - PLCC32 - CPU
Connections:
- net /CPU_EN renamed /~{PAR_PRGROM_EN}
- net /CPU_Game_EN renamed /~{GAME_PRGROM_EN}
- net /PPU_EN renamed /~{PAR_CHRROM_EN}
- net /PPU_Game_EN renamed /~{GAME_CHRROM_EN}
Changed lines of the file:
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@@
 	(net 81 "unconnected-(U1-OSC-Pad7)")
 	(net 82 "/FF.~{RST}")
-	(net 83 "/PPU_EN")
-	(net 84 "/CPU_EN")
+	(net 83 "/~{PAR_CHRROM_EN}")
+	(net 84 "/~{PAR_PRGROM_EN}")
 	(net 85 "/PPU_FF_CLK")
-	(net 86 "/PPU_Game_EN")
-	(net 87 "/CPU_Game_EN")
+	(net 86 "/~{GAME_CHRROM_EN}")
+	(net 87 "/~{GAME_PRGROM_EN}")
 	(net 88 "/CPU_FF_CLK")
 	(net 89 "/PPU_~{RD}.Game")
@@
 			)
 		)
-		(property "Value" "27C256 - PLCC32"
+		(property "Value" "27C256 - PLCC32 - CPU"
 			(at 0 1.5 0)
 			(unlocked yes)
@@
 			(size 0.6 1.5)
 			(layers "F.Cu" "F.Mask")
-			(net 87 "/CPU_Game_EN")
+			(net 87 "/~{GAME_PRGROM_EN}")
 			(pinfunction "D")
 			(pintype "input")
@@
 			(size 0.6 1.5)
 			(layers "F.Cu" "F.Mask")
-			(net 84 "/CPU_EN")
+			(net 84 "/~{PAR_PRGROM_EN}")
 			(pinfunction "Q")
 			(pintype "output")
@@
 			(size 0.6 1.5)
 			(layers "F.Cu" "F.Mask")
-			(net 87 "/CPU_Game_EN")
+			(net 87 "/~{GAME_PRGROM_EN}")
 			(pinfunction "~{Q}")
 			(pintype "output")
@@
 			(size 0.6 1.5)
 			(layers "F.Cu" "F.Mask")
-			(net 86 "/PPU_Game_EN")
+			(net 86 "/~{GAME_CHRROM_EN}")
 			(pinfunction "~{Q}")
 			(pintype "output")
@@
 			(size 0.6 1.5)
 			(layers "F.Cu" "F.Mask")
-			(net 83 "/PPU_EN")
+			(net 83 "/~{PAR_CHRROM_EN}")
 			(pinfunction "Q")
 			(pintype "output")
@@
 			(size 0.6 2.25)
 			(layers "F.Cu" "F.Mask")
-			(net 83 "/PPU_EN")
+			(net 83 "/~{PAR_CHRROM_EN}")
 			(pinfunction "I/O_2")
 			(pintype "bidirectional")
@@
 			(size 0.6 2.25)
 			(layers "F.Cu" "F.Mask")
-			(net 84 "/CPU_EN")
+			(net 84 "/~{PAR_PRGROM_EN}")
 			(pinfunction "I/O_4")
 			(pintype "bidirectional")
@@
 			(size 1.5 1.5)
 			(layers "F.Cu" "F.Mask")
-			(net 84 "/CPU_EN")
+			(net 84 "/~{PAR_PRGROM_EN}")
 			(pinfunction "K")
 			(pintype "passive")
@@
 			(size 0.6 1.5)
 			(layers "F.Cu" "F.Mask")
-			(net 84 "/CPU_EN")
+			(net 84 "/~{PAR_PRGROM_EN}")
 			(pintype "input")
 			(thermal_bridge_angle 45)
@@
 			(size 0.6 1.5)
 			(layers "F.Cu" "F.Mask")
-			(net 86 "/PPU_Game_EN")
+			(net 86 "/~{GAME_CHRROM_EN}")
 			(pintype "input")
 			(thermal_bridge_angle 45)
@@
 			(size 0.6 1.5)
 			(layers "F.Cu" "F.Mask")
-			(net 87 "/CPU_Game_EN")
+			(net 87 "/~{GAME_PRGROM_EN}")
 			(pintype "input")
 			(thermal_bridge_angle 45)
@@
 			(size 0.6 1.5)
 			(layers "F.Cu" "F.Mask")
-			(net 83 "/PPU_EN")
+			(net 83 "/~{PAR_CHRROM_EN}")
 			(pintype "input")
 			(thermal_bridge_angle 45)
@@
 			)
 		)
-		(property "Value" "27C256 - PLCC32"
+		(property "Value" "27C256 - PLCC32 - PPU"
 			(at 0 1.5 0)
 			(unlocked yes)
