File: NES3.kicad_sch (KiCad schematic)
At the start: 23 parts, among them SW1 SW_DPDT_x2, U2 27C256 - PLCC32, U3 74HC74, U4 74HC32, U5 27C256 - PLCC32, U7 HY6264ALJ

Commit message: Add files via upload
Parts:
- U2: value 27C256 - PLCC32 -> 27C256 - PLCC32 - PPU
- U5: value 27C256 - PLCC32 -> 27C256 - PLCC32 - CPU
Changed lines of the file:
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@@
 			)
 		)
-		(property "Value" "27C256 - PLCC32"
+		(property "Value" "27C256 - PLCC32 - PPU"
 			(at 136.8141 139.7 0)
 			(effects
@@
 			)
 		)
-		(property "Value" "27C256 - PLCC32"
+		(property "Value" "27C256 - PLCC32 - CPU"
 			(at 187.6141 139.7 0)
 			(effects

Commit message: Add files via upload
Connections:
- net CPU_EN renamed ~{PAR_PRGROM_EN}
- net CPU_Game_EN renamed ~{GAME_PRGROM_EN}
- net PPU_EN renamed ~{PAR_CHRROM_EN}
- net PPU_Game_EN renamed ~{GAME_CHRROM_EN}
Changed lines of the file:
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@@
 		)
 	)
-	(label "PPU_EN"
+	(label "~{PAR_CHRROM_EN}"
 		(at 346.71 74.93 0)
 		(effects
@@
 		)
 	)
-	(label "PPU_Game_EN"
+	(label "~{GAME_CHRROM_EN}"
 		(at 346.71 80.01 0)
 		(effects
@@
 		)
 	)
-	(label "CPU_Game_EN"
+	(label "~{GAME_PRGROM_EN}"
 		(at 302.26 80.01 0)
 		(effects
@@
 		)
 	)
-	(label "PPU_EN"
+	(label "~{PAR_CHRROM_EN}"
 		(at 337.82 45.72 180)
 		(effects
@@
 		)
 	)
-	(label "CPU_EN"
+	(label "~{PAR_PRGROM_EN}"
 		(at 299.72 199.39 0)
 		(effects
@@
 		)
 	)
-	(label "CPU_EN"
+	(label "~{PAR_PRGROM_EN}"
 		(at 302.26 74.93 0)
 		(effects
@@
 		)
 	)
-	(label "CPU_Game_EN"
+	(label "~{GAME_PRGROM_EN}"
 		(at 287.02 74.93 180)
 		(effects
@@
 		)
 	)
-	(label "PPU_Game_EN"
+	(label "~{GAME_CHRROM_EN}"
 		(at 337.82 29.21 180)
 		(effects
@@
 		)
 	)
-	(label "CPU_EN"
+	(label "~{PAR_PRGROM_EN}"
 		(at 293.37 30.48 180)
 		(effects
@@
 		)
 	)
-	(label "CPU_Game_EN"
+	(label "~{GAME_PRGROM_EN}"
 		(at 293.37 50.8 180)
 		(effects
@@
 		)
 	)
-	(label "PPU_EN"
+	(label "~{PAR_CHRROM_EN}"
 		(at 299.72 207.01 0)
 		(effects
@@
 		)
 	)
-	(label "CPU_EN"
+	(label "~{PAR_PRGROM_EN}"
 		(at 379.73 69.85 180)
 		(effects
